Commit message: feat:atom-w-p3

File: atom_urdf/urdf/atom_p3/atom_p3.urdf (robot description, URDF)
Before this commit: robot atom_p3, 39 links, 38 joints
Links:
- link head_pitch_link: geometry visual mesh filename=package://atom_urdf/meshes/atom_p3/head_pitch_link.STL
- link head_yaw_link: geometry visual mesh filename=package://atom_urdf/meshes/atom_p3/head_yaw_link.STL
- link left_ankle_pitch_link: geometry visual mesh filename=package://atom_urdf/meshes/atom_p3/left_ankle_pitch_link.STL
- link left_ankle_roll_link: geometry collision box size=0.24 0.08 0.02; visual mesh filename=package://atom_urdf/meshes/atom_p3/left_ankle_roll_link.STL
- link left_elbow_pitch_Link: geometry collision cylinder length=0.15 radius=0.038; visual mesh filename=package://atom_urdf/meshes/atom_p3/left_elbow_pitch_Link.STL
- link left_elbow_roll_Link: geometry visual mesh filename=package://atom_urdf/meshes/atom_p3/left_elbow_roll_Link.STL
- link left_hip_pitch_link: geometry visual mesh filename=package://atom_urdf/meshes/atom_p3/left_hip_pitch_link.STL
- link left_hip_roll_link: geometry collision cylinder length=0.35 radius=0.065; visual mesh filename=package://atom_urdf/meshes/atom_p3/left_hip_roll_link.STL
- link left_hip_yaw_link: geometry visual mesh filename=package://atom_urdf/meshes/atom_p3/left_hip_yaw_link.STL
- link left_knee_link: geometry collision cylinder length=0.3 radius=0.06; visual mesh filename=package://atom_urdf/meshes/atom_p3/left_knee_link.STL
- link left_shoulder_pitch_Link: geometry visual mesh filename=package://atom_urdf/meshes/atom_p3/left_shoulder_pitch_Link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
- link left_shoulder_roll_Link: geometry visual mesh filename=package://atom_urdf/meshes/atom_p3/left_shoulder_roll_Link.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
- link left_shoulder_yaw_Link: geometry collision cylinder length=0.24 radius=0.038; visual mesh filename=package://atom_urdf/meshes/atom_p3/left_shoulder_yaw_Link.S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
- link left_wrist_pitch_Link: geometry visual mesh filename=package://atom_urdf/meshes/atom_p3/left_wrist_pitch_Link.STL
- link left_wrist_yaw_Link: geometry collision sphere radius=0.05; visual mesh filename=package://atom_urdf/meshes/atom_p3/left_wrist_yaw_Link.STL
- link pelvis: geometry collision sphere radius=0.085; visual mesh filename=package://atom_urdf/meshes/atom_p3/pelvis.STL
- link right_ankle_pitch_link: geometry visual mesh filename=package://atom_urdf/meshes/atom_p3/right_ankle_pitch_link.S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
- link right_ankle_roll_link: geometry collision box size=0.24 0.08 0.02; visual mesh filename=package://atom_urdf/meshes/atom_p3/right_ankle_roll_link.STL
- link right_elbow_pitch_Link: geometry collision cylinder length=0.15 radius=0.038; visual mesh filename=package://atom_urdf/meshes/atom_p3/right_elbow_pitch_Link.S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
- link right_elbow_roll_Link: geometry visual mesh filename=package://atom_urdf/meshes/atom_p3/right_elbow_roll_Link.STL
- link right_hip_pitch_link: geometry visual mesh filename=package://atom_urdf/meshes/atom_p3/right_hip_pitch_link.STL
- link right_hip_roll_link: geometry collision cylinder length=0.35 radius=0.065; visual mesh filename=package://atom_urdf/meshes/atom_p3/right_hip_roll_link.STL
- link right_hip_yaw_link: geometry visual mesh filename=package://atom_urdf/meshes/atom_p3/right_hip_yaw_link.STL
- link right_knee_link: geometry collision cylinder length=0.3 radius=0.06; visual mesh filename=package://atom_urdf/meshes/atom_p3/right_knee_link.STL
- link right_shoulder_pitch_Link: geometry visual mesh filename=package://atom_urdf/meshes/atom_p3/right_shoulder_pitch_Lin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
- link right_shoulder_roll_Link: geometry visual mesh filename=package://atom_urdf/meshes/atom_p3/right_shoulder_roll_Link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
- link right_shoulder_yaw_Link: geometry collision cylinder length=0.24 radius=0.038; visual mesh filename=package://atom_urdf/meshes/atom_p3/right_shoulder_yaw_Link.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
- link right_wrist_pitch_Link: geometry visual mesh filename=package://atom_urdf/meshes/atom_p3/right_wrist_pitch_Link.S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
- link right_wrist_yaw_Link: geometry collision sphere radius=0.05; visual mesh filename=package://atom_urdf/meshes/atom_p3/right_wrist_yaw_Link.STL
- link torso_link: geometry collision box size=0.22 0.24 0.4; visual mesh filename=package://atom_urdf/meshes/atom_p3/torso_link.STL

File: atom_urdf/urdf/atom_w_p2/atom-w-p2.urdf (robot description, URDF)
Before this commit: robot atom_w_p2, 49 links, 48 joints
Links:
- link body_yaw_link: geometry collision mesh filename=package://atom_urdf/meshes/atom_w_p2/robot/body_yaw_link.STL; visual mesh filename=package://atom_urdf/meshes/atom_w_p2/robot/body_yaw_link.STL
- link chassis_link: geometry collision mesh filename=package://atom_urdf/meshes/atom_w_p2/robot/chassis_link.STL; visual mesh filename=package://atom_urdf/meshes/atom_w_p2/robot/chassis_link.STL
- link crus_pitch_link: geometry collision mesh filename=package://atom_urdf/meshes/atom_w_p2/robot/crus_pitch_link.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; visual mesh filename=package://atom_urdf/meshes/atom_w_p2/robot/crus_pitch_link.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
- link head_pitch_link: geometry collision mesh filename=package://atom_urdf/meshes/atom_w_p2/robot/head_pitch_link.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; visual mesh filename=package://atom_urdf/meshes/atom_w_p2/robot/head_pitch_link.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
- link head_yaw_link: geometry collision mesh filename=package://atom_urdf/meshes/atom_w_p2/robot/head_yaw_link.STL; visual mesh filename=package://atom_urdf/meshes/atom_w_p2/robot/head_yaw_link.STL
- link left_ag95_gripper_base_link: geometry collision mesh filename=package://atom_urdf/meshes/atom_w_p2/ag95/visual/base_link.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 scale=0.001 0.001 0.001; visual mesh filename=package://atom_urdf/meshes/atom_w_p2/ag95/visual/base_link.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 scale=0.001 0.001 0.001
- link left_ag95_gripper_finger1_finger_link: geometry collision mesh filename=package://atom_urdf/meshes/atom_w_p2/ag95/visual/rod_Link.S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 scale=0.001 0.001 0.001; visual mesh filename=package://atom_urdf/meshes/atom_w_p2/ag95/visual/rod_Link.S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 scale=0.001 0.001 0.001
- link left_ag95_gripper_finger1_finger_tip_link: geometry collision mesh filename=package://atom_urdf/meshes/atom_w_p2/ag95/visual/distal_pha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 scale=0.001 0.001 0.001; visual mesh filename=package://atom_urdf/meshes/atom_w_p2/ag95/visual/distal_pha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 scale=0.001 0.001 0.001
- link left_ag95_gripper_finger1_inner_knuckle_link: geometry collision mesh filename=package://atom_urdf/meshes/atom_w_p2/ag95/visual/proximal_p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 scale=0.001 0.001 0.001; visual mesh filename=package://atom_urdf/meshes/atom_w_p2/ag95/visual/proximal_p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 scale=0.001 0.001 0.001
- link left_ag95_gripper_finger1_knuckle_link: geometry collision mesh filename=package://atom_urdf/meshes/atom_w_p2/ag95/visual/crank_Link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 scale=0.001 0.001 0.001; visual mesh filename=package://atom_urdf/meshes/atom_w_p2/ag95/visual/crank_Link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 scale=0.001 0.001 0.001
- link left_ag95_gripper_finger2_finger_link: geometry collision mesh filename=package://atom_urdf/meshes/atom_w_p2/ag95/visual/rod_Link.S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 scale=0.001 0.001 0.001; visual mesh filename=package://atom_urdf/meshes/atom_w_p2/ag95/visual/rod_Link.S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 scale=0.001 0.001 0.001
- link left_ag95_gripper_finger2_finger_tip_link: geometry collision mesh filename=package://atom_urdf/meshes/atom_w_p2/ag95/visual/distal_pha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 scale=0.001 0.001 0.001; visual mesh filename=package://atom_urdf/meshes/atom_w_p2/ag95/visual/distal_pha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 scale=0.001 0.001 0.001
- link left_ag95_gripper_finger2_inner_knuckle_link: geometry collision mesh filename=package://atom_urdf/meshes/atom_w_p2/ag95/visual/proximal_p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 scale=0.001 0.001 0.001; visual mesh filename=package://atom_urdf/meshes/atom_w_p2/ag95/visual/proximal_p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 scale=0.001 0.001 0.001
- link left_ag95_gripper_finger2_knuckle_link: geometry collision mesh filename=package://atom_urdf/meshes/atom_w_p2/ag95/visual/crank_Link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 scale=0.001 0.001 0.001; visual mesh filename=package://atom_urdf/meshes/atom_w_p2/ag95/visual/crank_Link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 scale=0.001 0.001 0.001
- link left_camera_bracket_visual_link: geometry collision mesh filename=package://atom_urdf/meshes/atom_w_p2/camera_bracket/camera_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; visual mesh filename=package://atom_urdf/meshes/atom_w_p2/camera_bracket/camera_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
- link left_elbow_pitch_link: geometry collision mesh filename=package://atom_urdf/meshes/atom_w_p2/robot/left_elbow_pitch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; visual mesh filename=package://atom_urdf/meshes/atom_w_p2/robot/left_elbow_pitch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
- link left_elbow_roll_link: geometry collision mesh filename=package://atom_urdf/meshes/atom_w_p2/robot/left_elbow_roll_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; visual mesh filename=package://atom_urdf/meshes/atom_w_p2/robot/left_elbow_roll_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
- link left_flange_visual_link: geometry visual mesh filename=package://atom_urdf/meshes/atom_w_p2/flange/flange_0518_fix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
- link left_shoulder_pitch_link: geometry collision mesh filename=package://atom_urdf/meshes/atom_w_p2/robot/left_shoulder_pi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; visual mesh filename=package://atom_urdf/meshes/atom_w_p2/robot/left_shoulder_pi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
- link left_shoulder_roll_link: geometry collision mesh filename=package://atom_urdf/meshes/atom_w_p2/robot/left_shoulder_ro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; visual mesh filename=package://atom_urdf/meshes/atom_w_p2/robot/left_shoulder_ro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
- link left_shoulder_yaw_link: geometry collision mesh filename=package://atom_urdf/meshes/atom_w_p2/robot/left_shoulder_ya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; visual mesh filename=package://atom_urdf/meshes/atom_w_p2/robot/left_shoulder_ya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
- link left_whell_pitch_Link: geometry collision mesh filename=package://atom_urdf/meshes/atom_w_p2/wheels/left_whell_pitc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; visual mesh filename=package://atom_urdf/meshes/atom_w_p2/wheels/left_whell_pitc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
- link left_wrist_pitch_link: geometry collision mesh filename=package://atom_urdf/meshes/atom_w_p2/robot/left_wrist_pitch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; visual mesh filename=package://atom_urdf/meshes/atom_w_p2/robot/left_wrist_pitch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
- link left_wrist_yaw_link: geometry collision mesh filename=package://atom_urdf/meshes/atom_w_p2/robot/left_wrist_yaw_l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; visual mesh filename=package://atom_urdf/meshes/atom_w_p2/robot/left_wrist_yaw_l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
- link plevis_pitch_link: geometry collision mesh filename=package://atom_urdf/meshes/atom_w_p2/robot/plevis_pitch_lin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; visual mesh filename=package://atom_urdf/meshes/atom_w_p2/robot/plevis_pitch_lin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
- link right_ag95_gripper_base_link: geometry collision mesh filename=package://atom_urdf/meshes/atom_w_p2/ag95/visual/base_link.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 scale=0.001 0.001 0.001; visual mesh filename=package://atom_urdf/meshes/atom_w_p2/ag95/visual/base_link.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 scale=0.001 0.001 0.001
- link right_ag95_gripper_finger1_finger_link: geometry collision mesh filename=package://atom_urdf/meshes/atom_w_p2/ag95/visual/rod_Link.S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 scale=0.001 0.001 0.001; visual mesh filename=package://atom_urdf/meshes/atom_w_p2/ag95/visual/rod_Link.S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 scale=0.001 0.001 0.001
- link right_ag95_gripper_finger1_finger_tip_link: geometry collision mesh filename=package://atom_urdf/meshes/atom_w_p2/ag95/visual/distal_pha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 scale=0.001 0.001 0.001; visual mesh filename=package://atom_urdf/meshes/atom_w_p2/ag95/visual/distal_pha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 scale=0.001 0.001 0.001
- link right_ag95_gripper_finger1_inner_knuckle_link: geometry collision mesh filename=package://atom_urdf/meshes/atom_w_p2/ag95/visual/proximal_p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 scale=0.001 0.001 0.001; visual mesh filename=package://atom_urdf/meshes/atom_w_p2/ag95/visual/proximal_p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 scale=0.001 0.001 0.001
- link right_ag95_gripper_finger1_knuckle_link: geometry collision mesh filename=package://atom_urdf/meshes/atom_w_p2/ag95/visual/crank_Link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 scale=0.001 0.001 0.001; visual mesh filename=package://atom_urdf/meshes/atom_w_p2/ag95/visual/crank_Link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 scale=0.001 0.001 0.001
- link right_ag95_gripper_finger2_finger_link: geometry collision mesh filename=package://atom_urdf/meshes/atom_w_p2/ag95/visual/rod_Link.S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 scale=0.001 0.001 0.001; visual mesh filename=package://atom_urdf/meshes/atom_w_p2/ag95/visual/rod_Link.S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 scale=0.001 0.001 0.001
- link right_ag95_gripper_finger2_finger_tip_link: geometry collision mesh filename=package://atom_urdf/meshes/atom_w_p2/ag95/visual/distal_pha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 scale=0.001 0.001 0.001; visual mesh filename=package://atom_urdf/meshes/atom_w_p2/ag95/visual/distal_pha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 scale=0.001 0.001 0.001
- link right_ag95_gripper_finger2_inner_knuckle_link: geometry collision mesh filename=package://atom_urdf/meshes/atom_w_p2/ag95/visual/proximal_p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 scale=0.001 0.001 0.001; visual mesh filename=package://atom_urdf/meshes/atom_w_p2/ag95/visual/proximal_p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 scale=0.001 0.001 0.001
- link right_ag95_gripper_finger2_knuckle_link: geometry collision mesh filename=package://atom_urdf/meshes/atom_w_p2/ag95/visual/crank_Link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 scale=0.001 0.001 0.001; visual mesh filename=package://atom_urdf/meshes/atom_w_p2/ag95/visual/crank_Link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 scale=0.001 0.001 0.001
- link right_camera_bracket_visual_link: geometry collision mesh filename=package://atom_urdf/meshes/atom_w_p2/camera_bracket/camera_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; visual mesh filename=package://atom_urdf/meshes/atom_w_p2/camera_bracket/camera_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
- link right_elbow_pitch_link: geometry collision mesh filename=package://atom_urdf/meshes/atom_w_p2/robot/right_elbow_pitc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; visual mesh filename=package://atom_urdf/meshes/atom_w_p2/robot/right_elbow_pitc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
- link right_elbow_roll_link: geometry collision mesh filename=package://atom_urdf/meshes/atom_w_p2/robot/right_elbow_roll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; visual mesh filename=package://atom_urdf/meshes/atom_w_p2/robot/right_elbow_roll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
- link right_flange_visual_link: geometry visual mesh filename=package://atom_urdf/meshes/atom_w_p2/flange/flange_0518_fix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
- link right_shoulder_pitch_link: geometry collision mesh filename=package://atom_urdf/meshes/atom_w_p2/robot/right_shoulder_p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; visual mesh filename=package://atom_urdf/meshes/atom_w_p2/robot/right_shoulder_p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
- link right_shoulder_roll_link: geometry collision mesh filename=package://atom_urdf/meshes/atom_w_p2/robot/right_shoulder_r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; visual mesh filename=package://atom_urdf/meshes/atom_w_p2/robot/right_shoulder_r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
- link right_shoulder_yaw_link: geometry collision mesh filename=package://atom_urdf/meshes/atom_w_p2/robot/right_shoulder_y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; visual mesh filename=package://atom_urdf/meshes/atom_w_p2/robot/right_shoulder_y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
- link right_whell_pitch_Link: geometry collision mesh filename=package://atom_urdf/meshes/atom_w_p2/wheels/right_whell_pit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; visual mesh filename=package://atom_urdf/meshes/atom_w_p2/wheels/right_whell_pit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
- link right_wrist_pitch_link: geometry collision mesh filename=package://atom_urdf/meshes/atom_w_p2/robot/right_wrist_pitc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; visual mesh filename=package://atom_urdf/meshes/atom_w_p2/robot/right_wrist_pitc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
- link right_wrist_yaw_link: geometry collision mesh filename=package://atom_urdf/meshes/atom_w_p2/robot/right_wrist_yaw_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; visual mesh filename=package://atom_urdf/meshes/atom_w_p2/robot/right_wrist_yaw_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
- link thigh_pitch_link: geometry collision mesh filename=package://atom_urdf/meshes/atom_w_p2/robot/thigh_pitch_link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; visual mesh filename=package://atom_urdf/meshes/atom_w_p2/robot/thigh_pitch_link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

File: atom_urdf/urdf/atom_w_p3/atom-w-p3.urdf (robot description, URDF)
Before this commit: robot atom_w_p3, 23 links, 22 joints
Links:
- link calf_pitch_link: geometry collision mesh filename=package://atom_urdf/meshes/atom_w_p3/calf_pitch_link.STL; visual mesh filename=package://atom_urdf/meshes/atom_w_p3/calf_pitch_link.STL
- link chassis: geometry collision mesh filename=package://atom_urdf/meshes/atom_w_p3/chassis.STL; visual mesh filename=package://atom_urdf/meshes/atom_w_p3/chassis.STL
- link head_pitch_link: geometry collision mesh filename=package://atom_urdf/meshes/atom_w_p3/head_pitch_link.STL; visual mesh filename=package://atom_urdf/meshes/atom_w_p3/head_pitch_link.STL
- link head_yaw_link: geometry collision mesh filename=package://atom_urdf/meshes/atom_w_p3/head_yaw_link.STL; visual mesh filename=package://atom_urdf/meshes/atom_w_p3/head_yaw_link.STL
- link left_elbow_pitch_Link: geometry collision mesh filename=package://atom_urdf/meshes/atom_w_p3/left_elbow_pitch_Link.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; visual mesh filename=package://atom_urdf/meshes/atom_w_p3/left_elbow_pitch_Link.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
- link left_elbow_roll_Link: geometry collision mesh filename=package://atom_urdf/meshes/atom_w_p3/left_elbow_roll_Link.S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; visual mesh filename=package://atom_urdf/meshes/atom_w_p3/left_elbow_roll_Link.S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
- link left_shoulder_pitch_Link: geometry collision mesh filename=package://atom_urdf/meshes/atom_w_p3/left_shoulder_pitch_Li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; visual mesh filename=package://atom_urdf/meshes/atom_w_p3/left_shoulder_pitch_Li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
- link left_shoulder_roll_Link: geometry collision mesh filename=package://atom_urdf/meshes/atom_w_p3/left_shoulder_roll_Lin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; visual mesh filename=package://atom_urdf/meshes/atom_w_p3/left_shoulder_roll_Lin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
- link left_shoulder_yaw_Link: geometry collision mesh filename=package://atom_urdf/meshes/atom_w_p3/left_shoulder_yaw_Link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; visual mesh filename=package://atom_urdf/meshes/atom_w_p3/left_shoulder_yaw_Link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
- link left_wheel_link: geometry collision mesh filename=package://atom_urdf/meshes/atom_w_p3/left_wheel_link.STL; visual mesh filename=package://atom_urdf/meshes/atom_w_p3/left_wheel_link.STL
- link left_wirst_pitch_Link: geometry collision mesh filename=package://atom_urdf/meshes/atom_w_p3/left_wirst_pitch_Link.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; visual mesh filename=package://atom_urdf/meshes/atom_w_p3/left_wirst_pitch_Link.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
- link left_wirst_yaw_Link: geometry collision mesh filename=package://atom_urdf/meshes/atom_w_p3/left_wirst_yaw_Link.STL; visual mesh filename=package://atom_urdf/meshes/atom_w_p3/left_wirst_yaw_Link.STL
- link right_elbow_pitch_Link: geometry collision mesh filename=package://atom_urdf/meshes/atom_w_p3/right_elbow_pitch_Link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; visual mesh filename=package://atom_urdf/meshes/atom_w_p3/right_elbow_pitch_Link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
- link right_elbow_roll_Link: geometry collision mesh filename=package://atom_urdf/meshes/atom_w_p3/right_elbow_roll_Link.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; visual mesh filename=package://atom_urdf/meshes/atom_w_p3/right_elbow_roll_Link.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
- link right_shoulder_pitch_Link: geometry collision mesh filename=package://atom_urdf/meshes/atom_w_p3/right_shoulder_pitch_L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; visual mesh filename=package://atom_urdf/meshes/atom_w_p3/right_shoulder_pitch_L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
- link right_shoulder_roll_Link: geometry collision mesh filename=package://atom_urdf/meshes/atom_w_p3/right_shoulder_roll_Li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; visual mesh filename=package://atom_urdf/meshes/atom_w_p3/right_shoulder_roll_Li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
- link right_shoulder_yaw_Link: geometry collision mesh filename=package://atom_urdf/meshes/atom_w_p3/right_shoulder_yaw_Lin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; visual mesh filename=package://atom_urdf/meshes/atom_w_p3/right_shoulder_yaw_Lin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
- link right_wheel_link: geometry collision mesh filename=package://atom_urdf/meshes/atom_w_p3/right_wheel_link.STL; visual mesh filename=package://atom_urdf/meshes/atom_w_p3/right_wheel_link.STL
- link right_wirst_pitch_Link: geometry collision mesh filename=package://atom_urdf/meshes/atom_w_p3/right_wirst_pitch_Link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; visual mesh filename=package://atom_urdf/meshes/atom_w_p3/right_wirst_pitch_Link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
- link right_wirst_yaw_Link: geometry collision mesh filename=package://atom_urdf/meshes/atom_w_p3/right_wirst_yaw_Link.S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; visual mesh filename=package://atom_urdf/meshes/atom_w_p3/right_wirst_yaw_Link.S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
- link thigh_pitch_Link: geometry collision mesh filename=package://atom_urdf/meshes/atom_w_p3/thigh_pitch_Link.STL; visual mesh filename=package://atom_urdf/meshes/atom_w_p3/thigh_pitch_Link.STL
- link torso_yaw_Link: geometry collision mesh filename=package://atom_urdf/meshes/atom_w_p3/torso_yaw_Link.STL; visual mesh filename=package://atom_urdf/meshes/atom_w_p3/torso_yaw_Link.STL
- link waist_pitch_Link: geometry collision mesh filename=package://atom_urdf/meshes/atom_w_p3/waist_pitch_Link.STL; visual mesh filename=package://atom_urdf/meshes/atom_w_p3/waist_pitch_Link.STL
