Commit message: feat:atom-w-p3

File: atom_gazebo/urdf/atom_gazebo_control.xacro (robot description, xacro)
@@ -1,86 +1,22 @@
 <?xml version="1.0"?>
-<robot name="atom" xmlns:xacro="http://ros.org/wiki/xacro">
-  <!-- Include the base robot description -->
-  <xacro:include filename="$(find atom_urdf)/urdf/atom_p2/atom_gazebo.xacro" />
-  <!-- ROS2 Control Hardware Interface -->
-  <ros2_control name="AtomHardwareInterface" type="system">
+<robot name="atom_w_p3" xmlns:xacro="http://ros.org/wiki/xacro">
+  <xacro:include filename="$(find atom_urdf)/urdf/atom_w_p3/atom_w_p3.xacro" />
+  <ros2_control name="AtomWP3HardwareInterface" type="system">
     <hardware>
       <plugin>gazebo_ros2_control/GazeboSystem</plugin>
     </hardware>
-    <!-- Left leg joints -->
-    <joint name="leg_l1_joint">
-      <command_interface name="effort"/>
+    <joint name="left_wheel_joint">
+      <command_interface name="velocity"/>
       <state_interface name="position"/>
       <state_interface name="velocity"/>
       <state_interface name="effort"/>
     </joint>
-    <joint name="leg_l2_joint">
-      <command_interface name="effort"/>
+    <joint name="right_wheel_joint">
+      <command_interface name="velocity"/>
       <state_interface name="position"/>
       <state_interface name="velocity"/>
       <state_interface name="effort"/>
     </joint>
-    <joint name="leg_l3_joint">
-      <command_interface name="effort"/>
-      <state_interface name="position"/>
-      <state_interface name="velocity"/>
-      <state_interface name="effort"/>
-    </joint>
-    <joint name="leg_l4_joint">
-      <command_interface name="effort"/>
-      <state_interface name="position"/>
-      <state_interface name="velocity"/>
-      <state_interface name="effort"/>
-    </joint>
-    <joint name="leg_l5_joint">
-      <command_interface name="effort"/>
-      <state_interface name="position"/>
-      <state_interface name="velocity"/>
-      <state_interface name="effort"/>
-    </joint>
-    <joint name="leg_l6_joint">
-      <command_interface name="effort"/>
-      <state_interface name="position"/>
-      <state_interface name="velocity"/>
-      <state_interface name="effort"/>
-    </joint>
-    <!-- Right leg joints -->
-    <joint name="leg_r1_joint">
-      <command_interface name="effort"/>
-      <state_interface name="position"/>
-      <state_interface name="velocity"/>
-      <state_interface name="effort"/>
-    </joint>
-    <joint name="leg_r2_joint">
-      <command_interface name="effort"/>
-      <state_interface name="position"/>
-      <state_interface name="velocity"/>
-      <state_interface name="effort"/>
-    </joint>
-    <joint name="leg_r3_joint">
-      <command_interface name="effort"/>
-      <state_interface name="position"/>
-      <state_interface name="velocity"/>
-      <state_interface name="effort"/>
-    </joint>
-    <joint name="leg_r4_joint">
-      <command_interface name="effort"/>
-      <state_interface name="position"/>
-      <state_interface name="velocity"/>
-      <state_interface name="effort"/>
-    </joint>
-    <joint name="leg_r5_joint">
-      <command_interface name="effort"/>
-      <state_interface name="position"/>
-      <state_interface name="velocity"/>
-      <state_interface name="effort"/>
-    </joint>
-    <joint name="leg_r6_joint">
-      <command_interface name="effort"/>
-      <state_interface name="position"/>
-      <state_interface name="velocity"/>
-      <state_interface name="effort"/>
-    </joint>
-    <joint name="torso_joint">
+    <joint name="calf_pitch_joint">
       <command_interface name="position"/>
       <state_interface name="position"/>
@@ -88,6 +24,29 @@
       <state_interface name="effort"/>
     </joint>
-    <!-- Left arm joints -->
-    <joint name="left_shoulder_yaw_joint">
+    <joint name="thigh_pitch_joint">
+      <command_interface name="position"/>
+      <state_interface name="position"/>
+      <state_interface name="velocity"/>
+      <state_interface name="effort"/>
+    </joint>
+    <joint name="waist_pitch_joint">
+      <command_interface name="position"/>
+      <state_interface name="position"/>
+      <state_interface name="velocity"/>
+      <state_interface name="effort"/>
+    </joint>
+    <joint name="torso_yaw_joint">
+      <command_interface name="position"/>
+      <state_interface name="position"/>
+      <state_interface name="velocity"/>
+      <state_interface name="effort"/>
+    </joint>
+    <joint name="head_yaw_joint">
+      <command_interface name="position"/>
+      <state_interface name="position"/>
+      <state_interface name="velocity"/>
+      <state_interface name="effort"/>
+    </joint>
+    <joint name="head_pitch_joint">
       <command_interface name="position"/>
       <state_interface name="position"/>
@@ -107,4 +66,10 @@
       <state_interface name="effort"/>
     </joint>
+    <joint name="left_shoulder_yaw_joint">
+      <command_interface name="position"/>
+      <state_interface name="position"/>
+      <state_interface name="velocity"/>
+      <state_interface name="effort"/>
+    </joint>
     <joint name="left_elbow_pitch_joint">
       <command_interface name="position"/>
@@ -119,5 +84,5 @@
       <state_interface name="effort"/>
     </joint>
-    <joint name="left_wrist_pitch_joint">
+    <joint name="left_wirst_pitch_joint">
       <command_interface name="position"/>
       <state_interface name="position"/>
@@ -125,12 +90,5 @@
       <state_interface name="effort"/>
     </joint>
-    <joint name="left_wrist_yaw_joint">
-      <command_interface name="position"/>
-      <state_interface name="position"/>
-      <state_interface name="velocity"/>
-      <state_interface name="effort"/>
-    </joint>
-    <!-- Right arm joints -->
-    <joint name="right_shoulder_yaw_joint">
+    <joint name="left_wirst_yaw_joint">
       <command_interface name="position"/>
       <state_interface name="position"/>
@@ -150,4 +108,10 @@
       <state_interface name="effort"/>
     </joint>
+    <joint name="right_shoulder_yaw_joint">
+      <command_interface name="position"/>
+      <state_interface name="position"/>
+      <state_interface name="velocity"/>
+      <state_interface name="effort"/>
+    </joint>
     <joint name="right_elbow_pitch_joint">
       <command_interface name="position"/>
@@ -162,5 +126,5 @@
       <state_interface name="effort"/>
     </joint>
-    <joint name="right_wrist_pitch_joint">
+    <joint name="right_wirst_pitch_joint">
       <command_interface name="position"/>
       <state_interface name="position"/>
@@ -168,5 +132,5 @@
       <state_interface name="effort"/>
     </joint>
-    <joint name="right_wrist_yaw_joint">
+    <joint name="right_wirst_yaw_joint">
       <command_interface name="position"/>
       <state_interface name="position"/>
@@ -174,22 +138,8 @@
       <state_interface name="effort"/>
     </joint>
-    <!-- Head joints -->
-    <joint name="head_yaw_joint">
-      <command_interface name="effort"/>
-      <state_interface name="position"/>
-      <state_interface name="velocity"/>
-      <state_interface name="effort"/>
-    </joint>
-    <joint name="head_pitch_joint">
-      <command_interface name="effort"/>
-      <state_interface name="position"/>
-      <state_interface name="velocity"/>
-      <state_interface name="effort"/>
-    </joint>
   </ros2_control>
-  <!-- Gazebo ROS2 Control Plugin -->
   <gazebo>
     <plugin filename="libgazebo_ros2_control.so" name="gazebo_ros2_control">
-      <parameters>$(find atom_urdf)/config/atom_controllers.yaml</parameters>
+      <parameters>$(find atom_gazebo)/config/atom_w_p3_controllers.yaml</parameters>
       <ros>
         <remapping>/tf:=tf</remapping>
@@ -198,3 +148,35 @@
     </plugin>
   </gazebo>
+  <gazebo reference="left_wheel_link">
+    <mu1>0.8</mu1>
+    <mu2>0.8</mu2>
+    <kp>1000000.0</kp>
+    <kd>100.0</kd>
+    <material>Gazebo/DarkGrey</material>
+  </gazebo>
+  <gazebo reference="right_wheel_link">
+    <mu1>0.8</mu1>
+    <mu2>0.8</mu2>
+    <kp>1000000.0</kp>
+    <kd>100.0</kd>
+    <material>Gazebo/DarkGrey</material>
+  </gazebo>
+  <gazebo reference="imu_link">
+    <sensor name="imu_sensor" type="imu">
+      <always_on>true</always_on>
+      <update_rate>100</update_rate>
+      <imu>
+        <angular_velocity>
+          <x><noise type="gaussian" /><mean>0.0</mean><bias_stddev>0.001</bias_stddev></x>
+          <y><noise type="gaussian" /><mean>0.0</mean><bias_stddev>0.001</bias_stddev></y>
+          <z><noise type="gaussian" /><mean>0.0</mean><bias_stddev>0.001</bias_stddev></z>
+        </angular_velocity>
+        <linear_acceleration>
+          <x><noise type="gaussian" /><mean>0.0</mean><bias_stddev>0.001</bias_stddev></x>
+          <y><noise type="gaussian" /><mean>0.0</mean><bias_stddev>0.001</bias_stddev></y>
+          <z><noise type="gaussian" /><mean>0.0</mean><bias_stddev>0.001</bias_stddev></z>
+        </linear_acceleration>
+      </imu>
+    </sensor>
+  </gazebo>
 </robot>

File: atom_urdf/urdf/atom_w_p2/atom_w_p2.urdf (robot description, URDF)
Before this commit: robot atom_w_p2, 49 links, 48 joints
Links:
- added link imu_link
Joints:
- added joint imu_joint: type fixed, parent torso_link, child imu_link, origin xyz=0 0 -0.18 rpy=0 0 0

File: atom_urdf/urdf/atom_w_p3/atom_w_p3.xacro (robot description, xacro)
@@ -1,5 +1,4 @@
-<?xml version="1.0" encoding="utf-8"?>
-<robot
-  name="atom_w_p3">
+<?xml version="1.0"?>
+<robot name="atom" xmlns:xacro="http://ros.org/wiki/xacro">
   <link
     name="chassis">
@@ -24,5 +23,5 @@
       <geometry>
         <mesh
-          filename="package://atom_urdf/meshes/atom_w_p3/chassis.STL" />
+          filename="file://$(find atom_urdf)/meshes/atom_w_p3/chassis.STL" />
       </geometry>
       <material
@@ -38,5 +37,5 @@
       <geometry>
         <mesh
-          filename="package://atom_urdf/meshes/atom_w_p3/chassis.STL" />
+          filename="file://$(find atom_urdf)/meshes/atom_w_p3/chassis.STL" />
       </geometry>
     </collision>
@@ -64,5 +63,5 @@
       <geometry>
         <mesh
-          filename="package://atom_urdf/meshes/atom_w_p3/left_wheel_link.STL" />
+          filename="file://$(find atom_urdf)/meshes/atom_w_p3/left_wheel_link.STL" />
       </geometry>
       <material
@@ -78,5 +77,5 @@
       <geometry>
         <mesh
-          filename="package://atom_urdf/meshes/atom_w_p3/left_wheel_link.STL" />
+          filename="file://$(find atom_urdf)/meshes/atom_w_p3/left_wheel_link.STL" />
       </geometry>
     </collision>
@@ -120,5 +119,5 @@
       <geometry>
         <mesh
-          filename="package://atom_urdf/meshes/atom_w_p3/right_wheel_link.STL" />
+          filename="file://$(find atom_urdf)/meshes/atom_w_p3/right_wheel_link.STL" />
       </geometry>
       <material
@@ -134,5 +133,5 @@
       <geometry>
         <mesh
-          filename="package://atom_urdf/meshes/atom_w_p3/right_wheel_link.STL" />
+          filename="file://$(find atom_urdf)/meshes/atom_w_p3/right_wheel_link.STL" />
       </geometry>
     </collision>
@@ -176,19 +175,19 @@
       <geometry>
         <mesh
-          filename="package://atom_urdf/meshes/atom_w_p3/calf_pitch_link.STL" />
-      </geometry>
-      <material
-        name="">
-        <color
-          rgba="1 1 1 1" />
-      </material>
-    </visual>
-    <collision>
-      <origin
-        xyz="0 0 0"
-        rpy="0 0 0" />
-      <geometry>
-        <mesh
-          filename="package://atom_urdf/meshes/atom_w_p3/calf_pitch_link.STL" />
+          filename="file://$(find atom_urdf)/meshes/atom_w_p3/calf_pitch_link.STL" />
+      </geometry>
+      <material
+        name="">
+        <color
+          rgba="1 1 1 1" />
+      </material>
+    </visual>
+    <collision>
+      <origin
+        xyz="0 0 0"
+        rpy="0 0 0" />
+      <geometry>
+        <mesh
+          filename="file://$(find atom_urdf)/meshes/atom_w_p3/calf_pitch_link.STL" />
       </geometry>
     </collision>
@@ -234,19 +233,19 @@
       <geometry>
         <mesh
-          filename="package://atom_urdf/meshes/atom_w_p3/thigh_pitch_Link.STL" />
-      </geometry>
-      <material
-        name="">
-        <color
-          rgba="1 1 1 1" />
-      </material>
-    </visual>
-    <collision>
-      <origin
-        xyz="0 0 0"
-        rpy="0 0 0" />
-      <geometry>
-        <mesh
-          filename="package://atom_urdf/meshes/atom_w_p3/thigh_pitch_Link.STL" />
+          filename="file://$(find atom_urdf)/meshes/atom_w_p3/thigh_pitch_Link.STL" />
+      </geometry>
+      <material
+        name="">
+        <color
+          rgba="1 1 1 1" />
+      </material>
+    </visual>
+    <collision>
+      <origin
+        xyz="0 0 0"
+        rpy="0 0 0" />
+      <geometry>
+        <mesh
+          filename="file://$(find atom_urdf)/meshes/atom_w_p3/thigh_pitch_Link.STL" />
       </geometry>
     </collision>
@@ -292,19 +291,19 @@
       <geometry>
         <mesh
-          filename="package://atom_urdf/meshes/atom_w_p3/waist_pitch_Link.STL" />
-      </geometry>
-      <material
-        name="">
-        <color
-          rgba="1 1 1 1" />
-      </material>
-    </visual>
-    <collision>
-      <origin
-        xyz="0 0 0"
-        rpy="0 0 0" />
-      <geometry>
-        <mesh
-          filename="package://atom_urdf/meshes/atom_w_p3/waist_pitch_Link.STL" />
+          filename="file://$(find atom_urdf)/meshes/atom_w_p3/waist_pitch_Link.STL" />
+      </geometry>
+      <material
+        name="">
+        <color
+          rgba="1 1 1 1" />
+      </material>
+    </visual>
+    <collision>
+      <origin
+        xyz="0 0 0"
+        rpy="0 0 0" />
+      <geometry>
+        <mesh
+          filename="file://$(find atom_urdf)/meshes/atom_w_p3/waist_pitch_Link.STL" />
       </geometry>
     </collision>
@@ -350,19 +349,19 @@
       <geometry>
         <mesh
-          filename="package://atom_urdf/meshes/atom_w_p3/torso_yaw_Link.STL" />
-      </geometry>
-      <material
-        name="">
-        <color
-          rgba="1 1 1 1" />
-      </material>
-    </visual>
-    <collision>
-      <origin
-        xyz="0 0 0"
-        rpy="0 0 0" />
-      <geometry>
-        <mesh
-          filename="package://atom_urdf/meshes/atom_w_p3/torso_yaw_Link.STL" />
+          filename="file://$(find atom_urdf)/meshes/atom_w_p3/torso_yaw_Link.STL" />
+      </geometry>
+      <material
+        name="">
+        <color
+          rgba="1 1 1 1" />
+      </material>
+    </visual>
+    <collision>
+      <origin
+        xyz="0 0 0"
+        rpy="0 0 0" />
+      <geometry>
+        <mesh
+          filename="file://$(find atom_urdf)/meshes/atom_w_p3/torso_yaw_Link.STL" />
       </geometry>
     </collision>
@@ -408,5 +407,5 @@
       <geometry>
         <mesh
-          filename="package://atom_urdf/meshes/atom_w_p3/head_yaw_link.STL" />
+          filename="file://$(find atom_urdf)/meshes/atom_w_p3/head_yaw_link.STL" />
       </geometry>
       <material
@@ -422,5 +421,5 @@
       <geometry>
         <mesh
-          filename="package://atom_urdf/meshes/atom_w_p3/head_yaw_link.STL" />
+          filename="file://$(find atom_urdf)/meshes/atom_w_p3/head_yaw_link.STL" />
       </geometry>
     </collision>
@@ -466,5 +465,5 @@
       <geometry>
         <mesh
-          filename="package://atom_urdf/meshes/atom_w_p3/head_pitch_link.STL" />
+          filename="file://$(find atom_urdf)/meshes/atom_w_p3/head_pitch_link.STL" />
       </geometry>
       <material
@@ -480,5 +479,5 @@
       <geometry>
         <mesh
-          filename="package://atom_urdf/meshes/atom_w_p3/head_pitch_link.STL" />
+          filename="file://$(find atom_urdf)/meshes/atom_w_p3/head_pitch_link.STL" />
       </geometry>
     </collision>
@@ -524,19 +523,19 @@
       <geometry>
         <mesh
-          filename="package://atom_urdf/meshes/atom_w_p3/left_shoulder_pitch_Link.STL" />
-      </geometry>
-      <material
-        name="">
-        <color
-          rgba="1 1 1 1" />
-      </material>
-    </visual>
-    <collision>
-      <origin
-        xyz="0 0 0"
-        rpy="0 0 0" />
-      <geometry>
-        <mesh
-          filename="package://atom_urdf/meshes/atom_w_p3/left_shoulder_pitch_Link.STL" />
+          filename="file://$(find atom_urdf)/meshes/atom_w_p3/left_shoulder_pitch_Link.STL" />
+      </geometry>
+      <material
+        name="">
+        <color
+          rgba="1 1 1 1" />
+      </material>
+    </visual>
+    <collision>
+      <origin
+        xyz="0 0 0"
+        rpy="0 0 0" />
+      <geometry>
+        <mesh
+          filename="file://$(find atom_urdf)/meshes/atom_w_p3/left_shoulder_pitch_Link.STL" />
       </geometry>
     </collision>
@@ -582,19 +581,19 @@
       <geometry>
         <mesh
-          filename="package://atom_urdf/meshes/atom_w_p3/left_shoulder_roll_Link.STL" />
-      </geometry>
-      <material
-        name="">
-        <color
-          rgba="1 1 1 1" />
-      </material>
-    </visual>
-    <collision>
-      <origin
-        xyz="0 0 0"
-        rpy="0 0 0" />
-      <geometry>
-        <mesh
-          filename="package://atom_urdf/meshes/atom_w_p3/left_shoulder_roll_Link.STL" />
+          filename="file://$(find atom_urdf)/meshes/atom_w_p3/left_shoulder_roll_Link.STL" />
+      </geometry>
+      <material
+        name="">
+        <color
+          rgba="1 1 1 1" />
+      </material>
+    </visual>
+    <collision>
+      <origin
+        xyz="0 0 0"
+        rpy="0 0 0" />
+      <geometry>
+        <mesh
+          filename="file://$(find atom_urdf)/meshes/atom_w_p3/left_shoulder_roll_Link.STL" />
       </geometry>
     </collision>
@@ -640,19 +639,19 @@
       <geometry>
         <mesh
-          filename="package://atom_urdf/meshes/atom_w_p3/left_shoulder_yaw_Link.STL" />
-      </geometry>
-      <material
-        name="">
-        <color
-          rgba="1 1 1 1" />
-      </material>
-    </visual>
-    <collision>
-      <origin
-        xyz="0 0 0"
-        rpy="0 0 0" />
-      <geometry>
-        <mesh
-          filename="package://atom_urdf/meshes/atom_w_p3/left_shoulder_yaw_Link.STL" />
+          filename="file://$(find atom_urdf)/meshes/atom_w_p3/left_shoulder_yaw_Link.STL" />
+      </geometry>
+      <material
+        name="">
+        <color
+          rgba="1 1 1 1" />
+      </material>
+    </visual>
+    <collision>
+      <origin
+        xyz="0 0 0"
+        rpy="0 0 0" />
+      <geometry>
+        <mesh
+          filename="file://$(find atom_urdf)/meshes/atom_w_p3/left_shoulder_yaw_Link.STL" />
       </geometry>
     </collision>
@@ -698,19 +697,19 @@
       <geometry>
         <mesh
-          filename="package://atom_urdf/meshes/atom_w_p3/left_elbow_pitch_Link.STL" />
-      </geometry>
-      <material
-        name="">
-        <color
-          rgba="1 1 1 1" />
-      </material>
-    </visual>
-    <collision>
-      <origin
-        xyz="0 0 0"
-        rpy="0 0 0" />
-      <geometry>
-        <mesh
-          filename="package://atom_urdf/meshes/atom_w_p3/left_elbow_pitch_Link.STL" />
+          filename="file://$(find atom_urdf)/meshes/atom_w_p3/left_elbow_pitch_Link.STL" />
+      </geometry>
+      <material
+        name="">
+        <color
+          rgba="1 1 1 1" />
+      </material>
+    </visual>
+    <collision>
+      <origin
+        xyz="0 0 0"
+        rpy="0 0 0" />
+      <geometry>
+        <mesh
+          filename="file://$(find atom_urdf)/meshes/atom_w_p3/left_elbow_pitch_Link.STL" />
       </geometry>
     </collision>
@@ -743,32 +742,32 @@
         value="0.213" />
       <inertia
-        ixx="0"
+        ixx="0.000001"
         ixy="0"
         ixz="0"
-        iyy="0"
+        iyy="0.000001"
         iyz="0"
-        izz="0" />
-    </inertial>
-    <visual>
-      <origin
-        xyz="0 0 0"
-        rpy="0 0 0" />
-      <geometry>
-        <mesh
-          filename="package://atom_urdf/meshes/atom_w_p3/left_elbow_roll_Link.STL" />
-      </geometry>
-      <material
-        name="">
-        <color
-          rgba="1 1 1 1" />
-      </material>
-    </visual>
-    <collision>
-      <origin
-        xyz="0 0 0"
-        rpy="0 0 0" />
-      <geometry>
-        <mesh
-          filename="package://atom_urdf/meshes/atom_w_p3/left_elbow_roll_Link.STL" />
+        izz="0.000001" />
+    </inertial>
+    <visual>
+      <origin
+        xyz="0 0 0"
+        rpy="0 0 0" />
+      <geometry>
+        <mesh
+          filename="file://$(find atom_urdf)/meshes/atom_w_p3/left_elbow_roll_Link.STL" />
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